Commit message: Implement autonomous pick-and-place, HSV vision, Ackermann line-following, workspace mapping, and simulation fixes

File: src/ros2_ws/src/limo_cobot_bringup/urdf/gripper.xacro (robot description, xacro)
@@ -138,6 +138,18 @@
       <parent link="${parent_link}"/>
       <child link="${prefix}gripper_base"/>
-      <origin xyz="0 0 0.034" rpy="1.579 0 0"/>
-    </joint>
+      <origin xyz="0 0 0.034" rpy="1.579 0 1.5708"/>
+    </joint>
+    <joint name="${prefix}gripper_tcp_joint" type="fixed">
+      <parent link="${prefix}gripper_base"/>
+      <child link="${prefix}gripper_tcp"/>
+      <origin xyz="0 0.036 0" rpy="0 0 0"/>
+    </joint>
+    <link name="${prefix}gripper_tcp">
+      <inertial>
+        <mass value="0.001"/>
+        <origin xyz="0 0 0" rpy="0 0 0"/>
+        <inertia ixx="0.000001" ixy="0" ixz="0" iyy="0.000001" iyz="0" izz="0.000001"/>
+      </inertial>
+    </link>
     <joint name="${prefix}gripper_controller" type="revolute">
       <axis xyz="0 0 1"/>

Commit message: feat: implement limo-mycobot pickup pipeline, fix urdf meshes and prepare expert handover report

File: src/ros2_ws/src/limo_cobot_bringup/urdf/gripper.xacro (robot description, xacro)
@@ -5,5 +5,5 @@
       <visual>
         <geometry>
-          <mesh filename="package://mycobot_description/urdf/adaptive_gripper/gripper_base.dae"/>
+          <mesh filename="package://mycobot_description/meshes/mycobot_280/gripper_base.dae"/>
         </geometry>
         <origin xyz="0.0 0 -0.012" rpy="0 0 0"/>
@@ -11,5 +11,5 @@
       <collision>
         <geometry>
-          <mesh filename="package://mycobot_description/urdf/adaptive_gripper/gripper_base.dae"/>
+          <mesh filename="package://mycobot_description/meshes/mycobot_280/gripper_base.dae"/>
         </geometry>
         <origin xyz="0.0 0 -0.012" rpy="0 0 0"/>
@@ -24,5 +24,5 @@
       <visual>
         <geometry>
-          <mesh filename="package://mycobot_description/urdf/adaptive_gripper/gripper_left1.dae"/>
+          <mesh filename="package://mycobot_description/meshes/mycobot_280/gripper_left1.dae"/>
         </geometry>
         <origin xyz="0.039 -0.0133 -0.012" rpy="0 0 0"/>
@@ -30,5 +30,5 @@
       <collision>
         <geometry>
-          <mesh filename="package://mycobot_description/urdf/adaptive_gripper/gripper_left1.dae"/>
+          <mesh filename="package://mycobot_description/meshes/mycobot_280/gripper_left1.dae"/>
         </geometry>
         <origin xyz="0.039 -0.0133 -0.012" rpy="0 0 0"/>
@@ -43,5 +43,5 @@
       <visual>
         <geometry>
-          <mesh filename="package://mycobot_description/urdf/adaptive_gripper/gripper_left2.dae"/>
+          <mesh filename="package://mycobot_description/meshes/mycobot_280/gripper_left2.dae"/>
         </geometry>
         <origin xyz="0.005 -0.0195 -0.012" rpy="0 0 0"/>
@@ -49,5 +49,5 @@
       <collision>
         <geometry>
-          <mesh filename="package://mycobot_description/urdf/adaptive_gripper/gripper_left2.dae"/>
+          <mesh filename="package://mycobot_description/meshes/mycobot_280/gripper_left2.dae"/>
         </geometry>
         <origin xyz="0.005 -0.0195 -0.012" rpy="0 0 0"/>
@@ -62,5 +62,5 @@
       <visual>
         <geometry>
-          <mesh filename="package://mycobot_description/urdf/adaptive_gripper/gripper_left3.dae"/>
+          <mesh filename="package://mycobot_description/meshes/mycobot_280/gripper_left3.dae"/>
         </geometry>
         <origin xyz="0.012 0.0025 -0.012" rpy="0 0 0"/>
@@ -68,5 +68,5 @@
       <collision>
         <geometry>
-          <mesh filename="package://mycobot_description/urdf/adaptive_gripper/gripper_left3.dae"/>
+          <mesh filename="package://mycobot_description/meshes/mycobot_280/gripper_left3.dae"/>
         </geometry>
         <origin xyz="0.012 0.0025 -0.012" rpy="0 0 0"/>
@@ -81,5 +81,5 @@
       <visual>
         <geometry>
-          <mesh filename="package://mycobot_description/urdf/adaptive_gripper/gripper_right1.dae"/>
+          <mesh filename="package://mycobot_description/meshes/mycobot_280/gripper_right1.dae"/>
         </geometry>
         <origin xyz="-0.039 -0.0133 -0.012" rpy="0 0 0"/>
@@ -87,5 +87,5 @@
       <collision>
         <geometry>
-          <mesh filename="package://mycobot_description/urdf/adaptive_gripper/gripper_right1.dae"/>
+          <mesh filename="package://mycobot_description/meshes/mycobot_280/gripper_right1.dae"/>
         </geometry>
         <origin xyz="-0.039 -0.0133 -0.012" rpy="0 0 0"/>
@@ -100,5 +100,5 @@
       <visual>
         <geometry>
-          <mesh filename="package://mycobot_description/urdf/adaptive_gripper/gripper_right2.dae"/>
+          <mesh filename="package://mycobot_description/meshes/mycobot_280/gripper_right2.dae"/>
         </geometry>
         <origin xyz="-0.005 -0.0195 -0.012" rpy="0 0 0"/>
@@ -106,5 +106,5 @@
       <collision>
         <geometry>
-          <mesh filename="package://mycobot_description/urdf/adaptive_gripper/gripper_right2.dae"/>
+          <mesh filename="package://mycobot_description/meshes/mycobot_280/gripper_right2.dae"/>
         </geometry>
         <origin xyz="-0.005 -0.0195 -0.012" rpy="0 0 0"/>
@@ -119,5 +119,5 @@
       <visual>
         <geometry>
-          <mesh filename="package://mycobot_description/urdf/adaptive_gripper/gripper_right3.dae"/>
+          <mesh filename="package://mycobot_description/meshes/mycobot_280/gripper_right3.dae"/>
         </geometry>
         <origin xyz="-0.012 0.0025 -0.012" rpy="0 0 0"/>
@@ -125,5 +125,5 @@
       <collision>
         <geometry>
-          <mesh filename="package://mycobot_description/urdf/adaptive_gripper/gripper_right3.dae"/>
+          <mesh filename="package://mycobot_description/meshes/mycobot_280/gripper_right3.dae"/>
         </geometry>
         <origin xyz="-0.012 0.0025 -0.012" rpy="0 0 0"/>

File: src/ros2_ws/src/limo_cobot_bringup/urdf/limo_cobot_generated.urdf (robot description, URDF)
Before this commit: robot limo_cobot, 27 links, 26 joints
Links:
- removed link base_footprint
- added link depth_camera_frame_optical
- link base_link: mass 4.8 -> 4.34; geometry collision box size=0.19 0.31 0.12; visual mesh filename=/home/omar/Desktop/Thesis/src/ros2_ws/install/limo_car/shar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 scale=1.2 1.2 1.2
- link front_left_wheel_link: geometry collision cylinder length=0.045 radius=0.045; visual mesh filename=/home/omar/Desktop/Thesis/src/ros2_ws/install/limo_car/shar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 scale=1.2 1.2 1.2
- link front_right_wheel_link: geometry collision cylinder length=0.045 radius=0.045; visual mesh filename=/home/omar/Desktop/Thesis/src/ros2_ws/install/limo_car/shar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 scale=1.2 1.2 1.2
- link gripper_base: geometry collision mesh filename=package://mycobot_description/meshes/mycobot_280/gripper_ba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; visual mesh filename=package://mycobot_description/meshes/mycobot_280/gripper_ba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
- link gripper_left1: geometry collision mesh filename=package://mycobot_description/meshes/mycobot_280/gripper_le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; visual mesh filename=package://mycobot_description/meshes/mycobot_280/gripper_le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
- link gripper_left2: geometry collision mesh filename=package://mycobot_description/meshes/mycobot_280/gripper_le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; visual mesh filename=package://mycobot_description/meshes/mycobot_280/gripper_le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
- link gripper_left3: geometry collision mesh filename=package://mycobot_description/meshes/mycobot_280/gripper_le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; visual mesh filename=package://mycobot_description/meshes/mycobot_280/gripper_le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
- link gripper_right1: geometry collision mesh filename=package://mycobot_description/meshes/mycobot_280/gripper_ri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; visual mesh filename=package://mycobot_description/meshes/mycobot_280/gripper_ri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
- link gripper_right2: geometry collision mesh filename=package://mycobot_description/meshes/mycobot_280/gripper_ri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; visual mesh filename=package://mycobot_description/meshes/mycobot_280/gripper_ri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
- link gripper_right3: geometry collision mesh filename=package://mycobot_description/meshes/mycobot_280/gripper_ri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; visual mesh filename=package://mycobot_description/meshes/mycobot_280/gripper_ri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
- link joint1: geometry collision mesh filename=package://mycobot_description/meshes/mycobot_280/link1.dae; visual mesh filename=package://mycobot_description/meshes/mycobot_280/link1.dae
- link joint2: geometry collision mesh filename=package://mycobot_description/meshes/mycobot_280/link2.dae; visual mesh filename=package://mycobot_description/meshes/mycobot_280/link2.dae
- link joint3: geometry collision mesh filename=package://mycobot_description/meshes/mycobot_280/link3.dae; visual mesh filename=package://mycobot_description/meshes/mycobot_280/link3.dae
- link joint4: geometry collision mesh filename=package://mycobot_description/meshes/mycobot_280/link4.dae; visual mesh filename=package://mycobot_description/meshes/mycobot_280/link4.dae
- link joint5: geometry collision mesh filename=package://mycobot_description/meshes/mycobot_280/link5.dae; visual mesh filename=package://mycobot_description/meshes/mycobot_280/link5.dae
- link joint6: geometry collision mesh filename=package://mycobot_description/meshes/mycobot_280/link6.dae; visual mesh filename=package://mycobot_description/meshes/mycobot_280/link6.dae
- link joint6_flange: geometry collision mesh filename=package://mycobot_description/meshes/mycobot_280/link7.dae; visual mesh filename=package://mycobot_description/meshes/mycobot_280/link7.dae
- link rear_left_wheel_link: geometry collision cylinder length=0.045 radius=0.045; visual mesh filename=/home/omar/Desktop/Thesis/src/ros2_ws/install/limo_car/shar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 scale=1.2 1.2 1.2
- link rear_right_wheel_link: geometry collision cylinder length=0.045 radius=0.045; visual mesh filename=/home/omar/Desktop/Thesis/src/ros2_ws/install/limo_car/shar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 scale=1.2 1.2 1.2
Joints:
- removed joint base_joint
- added joint depth_camera_to_optical_joint: type fixed, parent depth_camera_link, child depth_camera_frame_optical, origin xyz=0 0 0 rpy=-1.570796 0 -1.570796 
- joint front_left_steer_joint: origin xyz=0.1 0.0875 -0.1 rpy=0 0 0 -> xyz=0.12 0.084 -0.1 rpy=0 0 0
- joint front_right_steer_joint: origin xyz=0.1 -0.0875 -0.1 rpy=3.14159 0 0 -> xyz=0.12 -0.084 -0.1 rpy=3.14159 0 0
- joint rear_left_wheel_joint: origin xyz=-0.1 0.0875 -0.1 rpy=0 0 0 -> xyz=-0.12 0.084 -0.1 rpy=0 0 0
- joint rear_right_wheel_joint: origin xyz=-0.1 -0.0875 -0.1 rpy=3.14159 0 0 -> xyz=-0.12 -0.084 -0.1 rpy=3.14159 0 0

File: src/ros2_ws/src/limo_cobot_bringup/urdf/mycobot_280_m5_gazebo.xacro (robot description, xacro)
@@ -26,5 +26,5 @@
       <visual>
         <geometry>
-          <mesh filename="package://mycobot_description/urdf/mycobot_280_m5/joint1.dae"/>
+          <mesh filename="package://mycobot_description/meshes/mycobot_280/link1.dae"/>
         </geometry>
         <origin xyz="0.0 0 0" rpy="0 0 -1.5708"/>
@@ -32,5 +32,5 @@
       <collision>
         <geometry>
-          <mesh filename="package://mycobot_description/urdf/mycobot_280_m5/joint1.dae"/>
+          <mesh filename="package://mycobot_description/meshes/mycobot_280/link1.dae"/>
         </geometry>
         <origin xyz="0.0 0 0" rpy="0 0 -1.5708"/>
@@ -45,5 +45,5 @@
       <visual>
         <geometry>
-          <mesh filename="package://mycobot_description/urdf/mycobot_280_m5/joint2.dae"/>
+          <mesh filename="package://mycobot_description/meshes/mycobot_280/link2.dae"/>
         </geometry>
         <origin xyz="0.0 0 -0.06096" rpy="0 0 -1.5708"/>
@@ -51,5 +51,5 @@
       <collision>
         <geometry>
-          <mesh filename="package://mycobot_description/urdf/mycobot_280_m5/joint2.dae"/>
+          <mesh filename="package://mycobot_description/meshes/mycobot_280/link2.dae"/>
         </geometry>
         <origin xyz="0.0 0 -0.06096" rpy="0 0 -1.5708"/>
@@ -64,5 +64,5 @@
       <visual>
         <geometry>
-          <mesh filename="package://mycobot_description/urdf/mycobot_280_m5/joint3.dae"/>
+          <mesh filename="package://mycobot_description/meshes/mycobot_280/link3.dae"/>
         </geometry>
         <origin xyz="0.0 0 0.03256" rpy="0 -1.5708 0"/>
@@ -70,5 +70,5 @@
       <collision>
         <geometry>
-          <mesh filename="package://mycobot_description/urdf/mycobot_280_m5/joint3.dae"/>
+          <mesh filename="package://mycobot_description/meshes/mycobot_280/link3.dae"/>
         </geometry>
         <origin xyz="0.0 0 0.03256" rpy="0 -1.5708 0"/>
@@ -83,5 +83,5 @@
       <visual>
         <geometry>
-          <mesh filename="package://mycobot_description/urdf/mycobot_280_m5/joint4.dae"/>
+          <mesh filename="package://mycobot_description/meshes/mycobot_280/link4.dae"/>
         </geometry>
         <origin xyz="0.0 0 0.03056" rpy="0 -1.5708 0"/>
@@ -89,5 +89,5 @@
       <collision>
         <geometry>
-          <mesh filename="package://mycobot_description/urdf/mycobot_280_m5/joint4.dae"/>
+          <mesh filename="package://mycobot_description/meshes/mycobot_280/link4.dae"/>
         </geometry>
         <origin xyz="0.0 0 0.03056" rpy="0 -1.5708 0"/>
@@ -102,5 +102,5 @@
       <visual>
         <geometry>
-          <mesh filename="package://mycobot_description/urdf/mycobot_280_m5/joint5.dae"/>
+          <mesh filename="package://mycobot_description/meshes/mycobot_280/link5.dae"/>
         </geometry>
         <origin xyz="0.0 0 -0.03356" rpy="-1.5708 0 0"/>
@@ -108,5 +108,5 @@
       <collision>
         <geometry>
-          <mesh filename="package://mycobot_description/urdf/mycobot_280_m5/joint5.dae"/>
+          <mesh filename="package://mycobot_description/meshes/mycobot_280/link5.dae"/>
         </geometry>
         <origin xyz="0.0 0 -0.03356" rpy="-1.5708 0 0"/>
@@ -121,5 +121,5 @@
       <visual>
         <geometry>
-          <mesh filename="package://mycobot_description/urdf/mycobot_280_m5/joint6.dae"/>
+          <mesh filename="package://mycobot_description/meshes/mycobot_280/link6.dae"/>
         </geometry>
         <origin xyz="0 0.00 -0.038" rpy="0 0 0"/>
@@ -127,5 +127,5 @@
       <collision>
         <geometry>
-          <mesh filename="package://mycobot_description/urdf/mycobot_280_m5/joint6.dae"/>
+          <mesh filename="package://mycobot_description/meshes/mycobot_280/link6.dae"/>
         </geometry>
         <origin xyz="0 0.00 -0.038" rpy="0 0 0"/>
@@ -140,5 +140,5 @@
       <visual>
         <geometry>
-          <mesh filename="package://mycobot_description/urdf/mycobot_280_m5/joint7.dae"/>
+          <mesh filename="package://mycobot_description/meshes/mycobot_280/link7.dae"/>
         </geometry>
         <origin xyz="0.0 0 -0.012" rpy="0 0 0"/>
@@ -146,5 +146,5 @@
       <collision>
         <geometry>
-          <mesh filename="package://mycobot_description/urdf/mycobot_280_m5/joint7.dae"/>
+          <mesh filename="package://mycobot_description/meshes/mycobot_280/link7.dae"/>
         </geometry>
         <origin xyz="0.0 0 -0.012" rpy="0 0 0"/>
@@ -303,35 +303,4 @@
         <state_interface name="velocity"/>
         <state_interface name="effort"/>
-      </joint>
-      <!-- Gripper passive/mimic joints (no command interfaces) -->
-      <joint name="${prefix}gripper_base_to_gripper_left2">
-        <param name="mimic">${prefix}gripper_controller</param>
-        <param name="multiplier">1.0</param>
-        <state_interface name="position"/>
-        <state_interface name="velocity"/>
-      </joint>
-      <joint name="${prefix}gripper_left3_to_gripper_left1">
-        <param name="mimic">${prefix}gripper_controller</param>
-        <param name="multiplier">-1.0</param>
-        <state_interface name="position"/>
-        <state_interface name="velocity"/>
-      </joint>
-      <joint name="${prefix}gripper_base_to_gripper_right3">
-        <param name="mimic">${prefix}gripper_controller</param>
-        <param name="multiplier">-1.0</param>
-        <state_interface name="position"/>
-        <state_interface name="velocity"/>
-      </joint>
-      <joint name="${prefix}gripper_base_to_gripper_right2">
-        <param name="mimic">${prefix}gripper_controller</param>
-        <param name="multiplier">-1.0</param>
-        <state_interface name="position"/>
-        <state_interface name="velocity"/>
-      </joint>
-      <joint name="${prefix}gripper_right3_to_gripper_right1">
-        <param name="mimic">${prefix}gripper_controller</param>
-        <param name="multiplier">1.0</param>
-        <state_interface name="position"/>
-        <state_interface name="velocity"/>
       </joint>
     </ros2_control>
