Commit message: feat: pick-and-place pipeline — Nav2 fixes, place table, map, dock drive
Navigation & costmap:
- Nav2 lifecycle manager delayed 6 s to fix map_server race condition
- Inflation radius 0.30→0.45m, cost_scaling_factor 3.0→2.5 (wider obstacle clearance)
- collision_monitor added to silence/activate lifecycle cycle so dock drive owns /cmd_vel
- station_a obstacle moved (-3.5,5)→(-5.0,7.5) to open 1.5m corridor for nav path
- RViz config switched to stable nav_monitor.rviz (no MoveIt panel = no segfault)

Place table:
- Moved place_table from (-2,0) to (-4,-2) — open area west of divider, clear nav path
- Static map updated: pickup_table and new place_table baked as occupied pixels
- NAV_PLACE_X/Y updated to (-4,-1.28), explicit PLACE_NAV_TO_DOCK=0.48 constant
- Place dock drive now uses absolute odom target y=-1.76 (robust vs Nav2 goal tolerance)

Grasp & weld:
- grasp_attacher: live TF lookup odom→gripper_tcp replaces stale startup pose capture
- smart_grasp.py: contact-based grasp detection (bumper + joint error fallback)
- Arm folds to travel pose at startup; ready pose kept for transit (box above LiDAR)

New scripts:
- smart_grasp.py — autonomous weld trigger on contact
- calib_pick.py, place_only_test.py, place_scenario.py — calibration/test utilities
- test_grasp_isolation.launch.py — isolated grasp test launch

Pre-navigate backup: robot reverses 0.6 m from pickup table before Nav2 plans
BACKUP_SEC reduced 4.0→2.5 s, nav timeout kept at 120 s

Co-Authored-By: Claude Sonnet 4.6 <noreply@anthropic.com>

File: src/ros2_ws/src/limo_cobot_bringup/urdf/gripper.xacro (robot description, xacro)
@@ -11,5 +11,5 @@
       <collision>
         <geometry>
-          <mesh filename="package://mycobot_description/meshes/mycobot_280/gripper_base.dae"/>
+          <box size="0.060 0.060 0.028"/>
         </geometry>
         <origin xyz="0.0 0 -0.012" rpy="0 0 0"/>
@@ -28,9 +28,10 @@
         <origin xyz="0.039 -0.0133 -0.012" rpy="0 0 0"/>
       </visual>
-      <collision>
-        <geometry>
-          <mesh filename="package://mycobot_description/meshes/mycobot_280/gripper_left1.dae"/>
-        </geometry>
-        <origin xyz="0.039 -0.0133 -0.012" rpy="0 0 0"/>
+      <!-- box replaces .dae collision: ODE ignores the mm unit tag, making the mesh 1000x too large -->
+      <collision>
+        <geometry>
+          <box size="0.036 0.013 0.024"/>
+        </geometry>
+        <origin xyz="0.037 -0.010 -0.012" rpy="0 0 0"/>
       </collision>
       <inertial>
@@ -49,5 +50,5 @@
       <collision>
         <geometry>
-          <mesh filename="package://mycobot_description/meshes/mycobot_280/gripper_left2.dae"/>
+          <box size="0.036 0.018 0.008"/>
         </geometry>
         <origin xyz="0.005 -0.0195 -0.012" rpy="0 0 0"/>
@@ -68,5 +69,5 @@
       <collision>
         <geometry>
-          <mesh filename="package://mycobot_description/meshes/mycobot_280/gripper_left3.dae"/>
+          <box size="0.005 0.036 0.036"/>
         </geometry>
         <origin xyz="0.012 0.0025 -0.012" rpy="0 0 0"/>
@@ -85,9 +86,10 @@
         <origin xyz="-0.039 -0.0133 -0.012" rpy="0 0 0"/>
       </visual>
-      <collision>
-        <geometry>
-          <mesh filename="package://mycobot_description/meshes/mycobot_280/gripper_right1.dae"/>
-        </geometry>
-        <origin xyz="-0.039 -0.0133 -0.012" rpy="0 0 0"/>
+      <!-- box replaces .dae collision: ODE ignores the mm unit tag, making the mesh 1000x too large -->
+      <collision>
+        <geometry>
+          <box size="0.013 0.024 0.036"/>
+        </geometry>
+        <origin xyz="-0.037 -0.010 -0.012" rpy="0 0 0"/>
       </collision>
       <inertial>
@@ -106,5 +108,5 @@
       <collision>
         <geometry>
-          <mesh filename="package://mycobot_description/meshes/mycobot_280/gripper_right2.dae"/>
+          <box size="0.018 0.008 0.036"/>
         </geometry>
         <origin xyz="-0.005 -0.0195 -0.012" rpy="0 0 0"/>
@@ -125,5 +127,5 @@
       <collision>
         <geometry>
-          <mesh filename="package://mycobot_description/meshes/mycobot_280/gripper_right3.dae"/>
+          <box size="0.036 0.036 0.005"/>
         </geometry>
         <origin xyz="-0.012 0.0025 -0.012" rpy="0 0 0"/>

File: src/ros2_ws/src/limo_ros2/limo_car/gazebo/ackermann.xacro (robot description, xacro)
@@ -2,5 +2,4 @@
 <!--Auto: Zhui Li-->
 <!--E-Mail: lz554113510@gmail.com -->
-<<<<<<< HEAD
 <!--Company: Institut fuer Intermodale Transport und Logistiksysteme in Technische Universitaet Braunschweig -->
 <!-- Description: Diese xacro-Datei basiert auf Regeln und definiert Funktionen durch xacro,
@@ -10,13 +9,4 @@
     <xacro:arg name="drive_mode" default="diff"/>
     <xacro:property name="drive_mode" value="$(arg drive_mode)"/>
-=======
-<!--Company: Institut für Intermodale Transport- und Logistiksysteme in Technische Universität Braunschweig -->
-<!-- Description: Diese xacro-Datei basiert auf Regeln und definiert Funktionen durch xacro,
-um die Erstellung der Struktur des Wagens in Ackerman-Type zu ermöglichen. Es liegen die Karosserie des kleinen Wagens,
-die Rädern und Steuerscharnier im vorderen Achse, und auch die hinten Rädern. Das ganze System ist als eine Makrofunktion
-dargestellt. Es erhält sich noch die Funktionen über Reglung für Lenkung und Bewegung, wie die in Gazebo realisiert werden.
-Es würde einfach in andere Datei angerufen werden. -->
-<robot name="limo_ackermann" xmlns:xacro="http://www.ros.org/wiki/xacro">
->>>>>>> origin/master
     <!-- ******************************** Paramenten zu definieren ************************************* -->
     <!-- *********************************************************************************************** -->
@@ -28,11 +18,6 @@
     <xacro:property name="base_y_size" value="0.31" />
     <xacro:property name="base_z_size" value="0.12" />
-<<<<<<< HEAD
     <xacro:property name="wheelbase" value="0.20"/>   <!-- LIMO PRO manual: wheel base 200mm -->
     <xacro:property name="track" value="0.175"/>      <!-- LIMO PRO manual: tread 175mm -->
-=======
-    <xacro:property name="wheelbase" value="0.24"/>
-    <xacro:property name="track" value="0.168"/>
->>>>>>> origin/master
     <xacro:property name="wheel_vertical_offset" value="-0.10" />
     <xacro:property name="wheel_mass" value="0.5" />
@@ -88,5 +73,4 @@
             </collision>
         </link>
-<<<<<<< HEAD
         <!-- diff drive: front-left wheel is a fixed mount (no steering) -->
         <joint name="${wheel_prefix}_steer_joint" type="fixed">
@@ -95,34 +79,9 @@
             <xacro:insert_block name="joint_pose"/>
         </joint>
-=======
-        <joint name="${wheel_prefix}_steer_joint" type="revolute">
-            <parent link="${parent_prefix}"/>
-            <child link="${wheel_prefix}_steer_link"/>
-            <xacro:insert_block name="joint_pose"/>
-            <axis xyz="0 0 1" />
-            <!-- Paramenten von Herstellern -->
-            <limit lower="-0.523598767" upper="0.523598767" effort="5" velocity="0.5" />
-            <dynamics damping="1.0" friction="2.0"/>
-        </joint>
-        <transmission name="${wheel_prefix}_hinge_trans" type="SimpleTransmission">
-            <type>transmission_interface/SimpleTransmission</type>
-            <actuator name="${wheel_prefix}_hinge_motor">
-                <hardwareInterface>hardware_interface/EffortJointInterface</hardwareInterface>
-                <mechanicalReduction>1</mechanicalReduction>
-            </actuator>
-            <joint name="${wheel_prefix}_steer_joint">
-                <hardwareInterface>hardware_interface/EffortJointInterface</hardwareInterface>
-            </joint>
-        </transmission>
->>>>>>> origin/master
         <link name="${wheel_prefix}_wheel_link">
             <visual>
                 <origin xyz="0 0 0" rpy="0 0 0" />
                 <geometry>
-<<<<<<< HEAD
                     <mesh filename="package://limo_car/meshes/limo_wheel.dae" scale="1.2 1.2 1.2"/>
-=======
-                    <mesh filename="$(find limo_car)/meshes/limo_wheel.dae" scale="1.2 1.2 1.2"/>
->>>>>>> origin/master
                 </geometry>
             </visual>
@@ -135,10 +94,7 @@
             <xacro:cylinder_inertial_matrix  m="${wheel_mass}" r="${wheel_radius}"  h="${wheel_length}" />
         </link>
-<<<<<<< HEAD
         <!-- differential drive: DRIVEN wheel. gazebo_ros_diff_drive spins this joint and the
              tyre friction grips the ground → REAL physics (gravity, traction, realistic odom).
              Left-side wheels spin about +Y. (Holonomic/mecanum version: ackermann_holonomic.xacro) -->
-=======
->>>>>>> origin/master
         <joint name="${wheel_prefix}_wheel_joint" type="continuous">
             <parent link="${wheel_prefix}_steer_link"/>
@@ -146,21 +102,6 @@
             <origin xyz="0 0 0" rpy="0 0 0" />
             <axis xyz="0 1 0"/>
-<<<<<<< HEAD
-            <dynamics damping="0.1" friction="0.1"/>
-        </joint>
-=======
-        </joint>
-        <transmission name="${wheel_prefix}_wheel_trans" type="SimpleTransmission">
-            <type>transmission_interface/SimpleTransmission</type>
-            <actuator name="${wheel_prefix}_wheel_motor">
-                <!-- Type für den Topic(Paramenten) -->
-                <hardwareInterface>hardware_interface/VelocityJointInterface</hardwareInterface>
-                <mechanicalReduction>1</mechanicalReduction>
-            </actuator>
-            <joint name="${wheel_prefix}_wheel_joint">
-                <hardwareInterface>hardware_interface/VelocityJointInterface</hardwareInterface>
-            </joint>
-        </transmission>
->>>>>>> origin/master
+            <dynamics damping="0.1" friction="0.1"/>
+        </joint>
     </xacro:macro>
     <!-- front right -->
@@ -185,5 +126,4 @@
             </collision>
         </link>
-<<<<<<< HEAD
         <!-- diff drive: front-right wheel is a fixed mount (no steering) -->
         <joint name="${wheel_prefix}_steer_joint" type="fixed">
@@ -192,33 +132,9 @@
             <xacro:insert_block name="joint_pose"/>
         </joint>
-=======
-        <joint name="${wheel_prefix}_steer_joint" type="revolute">
-            <parent link="${parent_prefix}"/>
-            <child link="${wheel_prefix}_steer_link"/>
-            <xacro:insert_block name="joint_pose"/>
-            <axis xyz="0 0 -1"/>
-            <limit lower="-0.523598767" upper="0.523598767" effort="5" velocity="0.5" />
-            <dynamics damping="1.0" friction="2.0"/>
-        </joint>
-        <transmission name="${wheel_prefix}_hinge_trans" type="SimpleTransmission">
-            <type>transmission_interface/SimpleTransmission</type>
-            <actuator name="${wheel_prefix}_hinge_motor">
-                <hardwareInterface>hardware_interface/EffortJointInterface</hardwareInterface>
-                <mechanicalReduction>1</mechanicalReduction>
-            </actuator>
-            <joint name="${wheel_prefix}_steer_joint">
-                <hardwareInterface>hardware_interface/EffortJointInterface</hardwareInterface>
-            </joint>
-        </transmission>
->>>>>>> origin/master
         <link name="${wheel_prefix}_wheel_link">
             <visual>
                 <origin xyz="0 0 0" rpy="0 0 0" />
                 <geometry>
-<<<<<<< HEAD
                     <mesh filename="package://limo_car/meshes/limo_wheel.dae" scale="1.2 1.2 1.2" />
-=======
-                    <mesh filename="$(find limo_car)/meshes/limo_wheel.dae" scale="1.2 1.2 1.2" />
->>>>>>> origin/master
                 </geometry>
             </visual>
@@ -231,5 +147,4 @@
             <xacro:cylinder_inertial_matrix  m="${wheel_mass}" r="${wheel_radius}"  h="${wheel_length}" />
         </link>
-<<<<<<< HEAD
         <!-- differential drive: DRIVEN wheel (see front-left note). Right-side spins about -Y. -->
         <joint name="${wheel_prefix}_wheel_joint" type="continuous">
@@ -240,23 +155,4 @@
             <dynamics damping="0.1" friction="0.1"/>
         </joint>
-=======
-        <joint name="${wheel_prefix}_wheel_joint" type="continuous">
-            <parent link="${wheel_prefix}_steer_link"/>
-            <child link="${wheel_prefix}_wheel_link"/>
-            <origin xyz="0 0 0" rpy="0 0  0" />
-            <axis xyz="0 -1 0"/>
-        </joint>
-        <transmission name="${wheel_prefix}_wheel_trans" type="SimpleTransmission">
-            <type>transmission_interface/SimpleTransmission</type>
-            <actuator name="${wheel_prefix}_wheel_motor">
-                <!-- Type für den Topic(Paramenten) -->
-                <hardwareInterface>hardware_interface/VelocityJointInterface</hardwareInterface>
-                <mechanicalReduction>1</mechanicalReduction>
-            </actuator>
-            <joint name="${wheel_prefix}_wheel_joint">
-                <hardwareInterface>hardware_interface/VelocityJointInterface</hardwareInterface>
-            </joint>
-        </transmission>
->>>>>>> origin/master
     </xacro:macro>
     <!-- *********************************************************************************************** -->
@@ -267,18 +163,10 @@
     Darstellungspostion in Simulation-Umgebung -->
     <xacro:macro name="limo_ackermann">
-<<<<<<< HEAD
         <link name="base_footprint"/>
-=======
-        <!-- <link name="base_footprint"/>
->>>>>>> origin/master
         <joint name="base_joint" type="fixed">
             <parent link="base_footprint"/>
             <child link="base_link"/>
             <origin xyz="0.0 0.0 0.15" rpy="0 0 0"/>
-<<<<<<< HEAD
-        </joint>
-=======
-        </joint> -->
->>>>>>> origin/master
+        </joint>
         <!-- herstellt base_link -->
         <link name="base_link">
@@ -287,5 +175,4 @@
                 <geometry>
                     <!-- Modell von Hersteller, aber es ist kleiner als realen Produkt, da die Skale vergrößert wird -->
-<<<<<<< HEAD
                     <mesh filename="package://limo_car/meshes/limo_base.stl" scale="0.0012 0.0012 0.0012" />
                 </geometry>
@@ -296,14 +183,4 @@
                 <geometry>
                     <mesh filename="package://limo_car/meshes/limo_base_collision_meters.stl" scale="1.0 1.0 1.0"/>
-=======
-                    <mesh filename="$(find limo_car)/meshes/limo_base.dae" scale="1.2 1.2 1.2" />
-                </geometry>
-            </visual>
-            <!-- Modell für physikalische Kollision zu modellieren. -->
-            <collision>
-                <origin xyz="0 0 0" rpy="0 0 0" />
-                <geometry>
-                    <box size="${base_x_size} ${base_y_size} ${base_z_size}"/>
->>>>>>> origin/master
                 </geometry>
             </collision>
@@ -320,9 +197,5 @@
                 <origin xyz="0 0 0" rpy="0 0 0" />
                 <geometry>
-<<<<<<< HEAD
                     <mesh filename="package://limo_car/meshes/limo_wheel.dae" scale="1.2 1.2 1.2"/>
-=======
-                    <mesh filename="$(find limo_car)/meshes/limo_wheel.dae" scale="1.2 1.2 1.2"/>
->>>>>>> origin/master
                 </geometry>
             </visual>
@@ -335,8 +208,5 @@
             <xacro:cylinder_inertial_matrix  m="${wheel_mass}" r="${wheel_radius}" h="${wheel_length}"/>
         </link>
-<<<<<<< HEAD
         <!-- differential drive: DRIVEN wheel (see front-left note). -->
-=======
->>>>>>> origin/master
         <joint name="rear_left_wheel_joint" type="continuous">
             <parent link="base_link"/>
@@ -344,29 +214,11 @@
             <origin xyz="${-wheelbase/2} ${track/2} ${wheel_vertical_offset}" rpy="0 0 0" />
             <axis xyz="0 1 0"/>
-<<<<<<< HEAD
-            <dynamics damping="0.1" friction="0.1"/>
-        </joint>
-=======
-        </joint>
-        <transmission name="rear_left_wheel_trans" type="SimpleTransmission">
-            <type>transmission_interface/SimpleTransmission</type>
-            <actuator name="rear_left_wheel_motor">
-                <hardwareInterface>hardware_interface/VelocityJointInterface</hardwareInterface>
-                <mechanicalReduction>1</mechanicalReduction>
-            </actuator>
-            <joint name="rear_left_wheel_joint">
-                <hardwareInterface>hardware_interface/VelocityJointInterface</hardwareInterface>
-            </joint>
-        </transmission>
->>>>>>> origin/master
+            <dynamics damping="0.1" friction="0.1"/>
+        </joint>
         <link name="rear_right_wheel_link">
             <visual>
                 <origin xyz="0 0 0" rpy="0 0 0" />
                 <geometry>
-<<<<<<< HEAD
                     <mesh filename="package://limo_car/meshes/limo_wheel.dae" scale="1.2 1.2 1.2"/>
-=======
-                    <mesh filename="$(find limo_car)/meshes/limo_wheel.dae" scale="1.2 1.2 1.2"/>
->>>>>>> origin/master
                 </geometry>
             </visual>
@@ -379,8 +231,5 @@
             <xacro:cylinder_inertial_matrix  m="${wheel_mass}" r="${wheel_radius}" h="${wheel_length}"/>
         </link>
-<<<<<<< HEAD
         <!-- differential drive: DRIVEN wheel (see front-left note). -->
-=======
->>>>>>> origin/master
         <joint name="rear_right_wheel_joint" type="continuous">
             <parent link="base_link"/>
@@ -388,20 +237,6 @@
             <origin xyz="${-wheelbase/2} ${-track/2} ${wheel_vertical_offset}" rpy="${M_PI} 0 0" />
             <axis xyz="0 -1 0"/>
-<<<<<<< HEAD
-            <dynamics damping="0.1" friction="0.1"/>
-        </joint>
-=======
-        </joint>
-        <transmission name="rear_right_wheel_trans" type="SimpleTransmission">
-            <type>transmission_interface/SimpleTransmission</type>
-            <actuator name="rear_right_wheel_motor">
-                <hardwareInterface>hardware_interface/VelocityJointInterface</hardwareInterface>
-                <mechanicalReduction>1</mechanicalReduction>
-            </actuator>
-            <joint name="rear_right_wheel_joint">
-                <hardwareInterface>hardware_interface/VelocityJointInterface</hardwareInterface>
-            </joint>
-        </transmission>
->>>>>>> origin/master
+            <dynamics damping="0.1" friction="0.1"/>
+        </joint>
         <!-- ruft Steuerscharnier mit vorderem Räder auf -->
         <xacro:limo_left_steering_hinge parent_prefix="base_link" wheel_prefix="front_left">
@@ -413,5 +248,4 @@
         <!-- ********************************** Kontrolle zu erstellen ************************************* -->
         <!-- *********************************************************************************************** -->
-<<<<<<< HEAD
         <!-- ── Differential drive (gazebo_ros_diff_drive) — REAL physics ──────────────
              Drives the 4 wheels as 2 pairs (left/right). cmd_vel.linear.x = forward,
@@ -438,26 +272,4 @@
                 <wheel_diameter>0.09</wheel_diameter>        <!-- 2 × 0.045 m radius -->
                 <wheel_diameter>0.09</wheel_diameter>
-=======
-        <gazebo>
-            <plugin name="gazebo_ros_control" filename="libgazebo_ros_control.so" />
-            <plugin name="ackermann_controller" filename="libgazebo_ros_ackermann_drive.so">
-                <update_rate>100</update_rate>
-                <front_left_joint>front_left_wheel_joint</front_left_joint>
-                <front_right_joint>front_right_wheel_joint</front_right_joint>
-                <rear_left_joint>rear_left_wheel_joint</rear_left_joint>
-                <rear_right_joint>rear_right_wheel_joint</rear_right_joint>
-                <left_steering_joint>front_left_steer_joint</left_steering_joint>
-                <right_steering_joint>front_right_steer_joint</right_steering_joint>
-                <steering_wheel_joint>/</steering_wheel_joint>
-                <left_steering_pid_gain>10000 100 10</left_steering_pid_gain>
-                <left_steering_i_rang>0 0</left_steering_i_rang>
-                <right_steering_pid_gain>10000 100 10</right_steering_pid_gain>
-                <right_steering_i_rang>0 0</right_steering_i_rang>
-                <linear_velocity_pid_gain>0.5 10 0.001</linear_velocity_pid_gain>
-                <linear_velocity_i_range>0 0</linear_velocity_i_range>
-                <max_steer>0.523598767</max_steer>
-                <wheel_separation>0.172</wheel_separation>
-                <wheel_diameter>0.09</wheel_diameter>
->>>>>>> origin/master
                 <max_wheel_torque>20</max_wheel_torque>
                 <max_wheel_acceleration>1.0</max_wheel_acceleration>
