Commit message: feat: pick-and-place pipeline — Nav2 fixes, place table, map, dock drive
Navigation & costmap:
- Nav2 lifecycle manager delayed 6 s to fix map_server race condition
- Inflation radius 0.30→0.45m, cost_scaling_factor 3.0→2.5 (wider obstacle clearance)
- collision_monitor added to silence/activate lifecycle cycle so dock drive owns /cmd_vel
- station_a obstacle moved (-3.5,5)→(-5.0,7.5) to open 1.5m corridor for nav path
- RViz config switched to stable nav_monitor.rviz (no MoveIt panel = no segfault)

Place table:
- Moved place_table from (-2,0) to (-4,-2) — open area west of divider, clear nav path
- Static map updated: pickup_table and new place_table baked as occupied pixels
- NAV_PLACE_X/Y updated to (-4,-1.28), explicit PLACE_NAV_TO_DOCK=0.48 constant
- Place dock drive now uses absolute odom target y=-1.76 (robust vs Nav2 goal tolerance)

Grasp & weld:
- grasp_attacher: live TF lookup odom→gripper_tcp replaces stale startup pose capture
- smart_grasp.py: contact-based grasp detection (bumper + joint error fallback)
- Arm folds to travel pose at startup; ready pose kept for transit (box above LiDAR)

New scripts:
- smart_grasp.py — autonomous weld trigger on contact
- calib_pick.py, place_only_test.py, place_scenario.py — calibration/test utilities
- test_grasp_isolation.launch.py — isolated grasp test launch

Pre-navigate backup: robot reverses 0.6 m from pickup table before Nav2 plans
BACKUP_SEC reduced 4.0→2.5 s, nav timeout kept at 120 s

Co-Authored-By: Claude Sonnet 4.6 <noreply@anthropic.com>

File: src/ros2_ws/src/limo_ros2/limo_car/gazebo/ackermann_with_sensor.xacro (robot description, xacro)
@@ -1,4 +1,3 @@
 <?xml version="1.0"?>
-<<<<<<< HEAD
 <robot name="limo_ackermann" xmlns:xacro="http://www.ros.org/wiki/xacro">
     <!-- use_camera:=false drops the GPU depth camera (driving/nav demos with the GUI),
@@ -6,24 +5,11 @@
     <xacro:arg name="use_camera" default="true"/>
     <xacro:property name="use_camera" value="$(arg use_camera)"/>
-=======
-<!--Auto: Zhui Li-->
-<!--E-Mail: lz554113510@gmail.com -->
-<!--Company: Institut für Intermodale Transport- und Logistiksysteme in Technische Universität Braunschweig -->
-<!-- Description: Diese xacro-Datei basiert auf Regeln und definiert Funktionen durch xacro,
-um die Erstellung der ganzen Struktur des Wagens in Ackerman-Type zu ermöglichen. Das Fahrzeuggrundmodell und
-andere Sensoren zusammengebaut werden und laden sie das Modell in Gazebo.-->
-<robot name="limo_ackermann" xmlns:xacro="http://www.ros.org/wiki/xacro">
->>>>>>> origin/master
     <xacro:include filename="$(find limo_car)/gazebo/ackermann.xacro" />
     <xacro:include filename="$(find limo_car)/gazebo/sensor.xacro" />
-<<<<<<< HEAD
     <!-- Instantiate the robot base -->
     <xacro:limo_ackermann />
-=======
->>>>>>> origin/master
     <!-- ************************* Laser ****************************** -->
     <xacro:gazebo_laser frame_prefix="laser" />
     <joint name="laser_joint" type="fixed">
-<<<<<<< HEAD
         <origin xyz="0.1236 0 -0.01" rpy="0 0 0"/>   <!-- realistic LIMO front-low mount; works now that the laser's own collision is 0.001 (was blinded by a 0.032 self-collision puck) -->
         <parent link="base_link"/>
@@ -39,17 +25,4 @@
         </joint>
     </xacro:if>
-=======
-        <origin xyz="0.1236 0 -0.01" rpy="0 0 0"/>
-        <parent link="base_link"/>
-        <child link="laser_link"/>
-    </joint>
-    <!-- ************************* Depth-camera *********************** -->
-    <xacro:gazebo_depth_camera frame_prefix="depth_camera" />
-    <joint name="depth_camera_joint" type="fixed">
-        <origin xyz="0.1 0 0.065" rpy="0 0 0"/>
-        <parent link="base_link"/>
-        <child link="depth_camera_link"/>
-    </joint>
->>>>>>> origin/master
     <!-- ************************* IMU ******************************** -->
     <xacro:gazebo_imu frame_prefix="imu" />
@@ -59,5 +32,4 @@
         <child link="imu_link"/>
     </joint>
-<<<<<<< HEAD
     <!-- ************************* MyCobot 280 Arm ************************ -->
     <xacro:include filename="$(find mycobot_description)/urdf/mycobot_280_m5/mycobot_280_m5.urdf" />
@@ -93,5 +65,3 @@
     <!-- ************************* ROS 2 Control ************************** -->
     <xacro:include filename="$(find limo_car)/gazebo/mycobot_ros2_control.xacro" />
-=======
->>>>>>> origin/master
 </robot>

File: src/ros2_ws/src/limo_ros2/limo_car/gazebo/sensor.xacro (robot description, xacro)
@@ -2,14 +2,7 @@
 <!-- Autor: Zhui Li -->
 <!--E-Mail: lz554113510@gmail.com -->
-<<<<<<< HEAD
 <!--Company: Institut fuer Intermodale Transport und Logistiksysteme in Technische Universitaet Braunschweig -->
 <!-- Description: Diese xacro-Datei basiert auf Regeln und definiert Funktionen durch xacro,
 um die Erstellung der weitere Simulation fuer Sensoren in Gazebo ermoeglichen. -->
-=======
-<!--Company: Institut für Intermodale Transport- und Logistiksysteme in Technische Universität Braunschweig -->
-<!-- Description: Diese xacro-Datei basiert auf Regeln und definiert Funktionen durch xacro,
-um die Erstellung der weitere Simulation für Sensoren in Gazebo ermöglichen. Es erhaltet die Makrofunktion für die
-realisierbar elektrische Komponente, also Sensoren aus Gazebo-Package. Diese Anteile konnte in anderen Datei benutzt werden. -->
->>>>>>> origin/master
 <robot name="limo_sensor" xmlns:xacro="http://www.ros.org/wiki/xacro">
     <!-- ******************************* Makrofunktion für Laser-Sensor ***************************** -->
@@ -41,9 +34,5 @@
                 <origin xyz="0 0 0" rpy="0 0 0"/>
                 <geometry>
-<<<<<<< HEAD
                     <cylinder radius="0.001" length="0.001"/>   <!-- shrunk from 0.032: a CPU ray sensor hits its own link collision, so the fat puck was blocking all beams -->
-=======
-                    <cylinder radius="0.032" length="0.016"/>
->>>>>>> origin/master
                 </geometry>
             </collision>
@@ -51,9 +40,5 @@
         <gazebo reference="${frame_prefix}_link">
             <sensor type="ray" name="laser_sensor">
-<<<<<<< HEAD
                 <visualize>true</visualize>
-=======
-                <visualize>false</visualize>
->>>>>>> origin/master
                 <update_rate>8</update_rate>
                 <ray>
@@ -62,5 +47,4 @@
                             <samples>720</samples>
                             <resolution>1</resolution>
-<<<<<<< HEAD
                             <min_angle>-2.09439510</min_angle> <!-- ±120° (240° forward arc). Rear 120° cut to avoid self-scanning the chassis/arm. Ref: limo_gazebo.gazebo in omaroped/workSPACELIMO. Original bad agent set this to ±180° (full 360°) which caused the robot to scan its own body. -->
                             <max_angle>2.09439510</max_angle>
@@ -70,13 +54,4 @@
                         <min>0.10</min>   <!-- 10cm minimum — filters chassis self-hits (6-7cm at ±108-120°); T-mini Pro real min is ~0.1m -->
                         <max>12.0</max>   <!-- EAI T-mini Pro: max 12 m -->
-=======
-                            <min_angle>-2.09439504</min_angle> <!-- Einheit in "rad", von Hersteller -->
-                            <max_angle>2.09439504</max_angle>
-                        </horizontal>
-                    </scan>
-                    <range>
-                        <min>0.2</min>
-                        <max>8.0</max>
->>>>>>> origin/master
                         <resolution>0.01</resolution>
                     </range>
@@ -94,9 +69,5 @@
                     </ros>
                     <output_type>sensor_msgs/LaserScan</output_type>
-<<<<<<< HEAD
                     <frame_name>${frame_prefix}_link</frame_name>
-=======
-                    <min_intensity>150.0</min_intensity>
->>>>>>> origin/master
                 </plugin>
             </sensor>
@@ -142,18 +113,8 @@
             <child link="depth_link"/>
         </joint>
-<<<<<<< HEAD
-=======
-        <link name="${frame_prefix}_frame_optical" />
-        <joint name="${frame_prefix}_to_optical_joint" type="fixed">
-            <origin xyz="0 0 0" rpy="-1.570796 0 -1.570796 "/>
-            <parent link="${frame_prefix}_link"/>
-            <child link="${frame_prefix}_frame_optical"/>
-        </joint>
->>>>>>> origin/master
         <gazebo reference="${frame_prefix}_link">
             <sensor name="sensor_camera" type="depth">
                 <pose>0.0 0.0 0.0 0.0 0.0 0.0</pose>
                 <always_on>true</always_on>
-<<<<<<< HEAD
                 <visualize>false</visualize>   <!-- hides the white camera frustum in Gazebo; camera still works/publishes. Set true to show it again -->
                 <update_rate>10.0</update_rate>
@@ -170,19 +131,4 @@
                         <near>0.15</near>
                         <far>3.0</far>   <!-- Orbbec DaBai depth max 3.0 m (was 8.0) -->
-=======
-                <visualize>true</visualize>
-                <update_rate>10.0</update_rate>
-                <camera name="head">
-                    <horizontal_fov>1.3962634</horizontal_fov> <!-- 60*pi/180 -->
-                    <!-- normalisieren die Form für Fotos -->
-                    <image>
-                        <width>640</width>
-                        <height>480</height>
-                        <format>R8G8B8</format>
-                    </image>
-                    <clip>
-                        <near>0.15</near>
-                        <far>8.0</far>
->>>>>>> origin/master
                     </clip>
                 </camera>
@@ -197,5 +143,4 @@
                     </ros>
                     <camera_name>${frame_prefix}</camera_name>
-<<<<<<< HEAD
                     <!-- Stamp images with depth_link, the actual optical frame that
                          exists in the TF tree (its joint applies the REP-103 optical
@@ -203,7 +148,4 @@
                          a real frame, so box_pose_estimator's TF lookup failed. -->
                     <frame_name>depth_link</frame_name>
-=======
-                    <frame_name>${frame_prefix}_frame_optical</frame_name>
->>>>>>> origin/master
                     <hack_baseline>0.07</hack_baseline>
                     <min_depth>0.001</min_depth>

File: src/ros2_ws/src/limo_ros2/limo_car/urdf/limo_ackerman_base.xacro (robot description, xacro)
@@ -11,9 +11,5 @@
     <!-- definiert Value -->
     <xacro:property name="M_PI" value="3.14159"/>
-<<<<<<< HEAD
     <xacro:property name="base_mass" value="2.1557"/>   <!-- base box only; LIMO PRO total mass ≈ 4.2 kg (verify link sum). Do NOT inflate this to fix base drift — that is a TEST-FIXTURE concern (base_pin), not a model property. -->
-=======
-    <xacro:property name="base_mass" value="2.1557"/>
->>>>>>> origin/master
     <xacro:property name="base_x_size" value="0.13" />
     <xacro:property name="base_y_size" value="0.12" />
@@ -23,9 +19,5 @@
 <!--    <xacro:property name="base_z_size" value="0.12" />-->
     <xacro:property name="wheelbase" value="0.2"/>
-<<<<<<< HEAD
     <xacro:property name="track" value="0.175"/>   <!-- LIMO PRO tread 175 mm (was 0.14) -->
-=======
-    <xacro:property name="track" value="0.14"/>
->>>>>>> origin/master
     <xacro:property name="wheel_vertical_offset" value="-0.100998" />
     <xacro:property name="wheel_mass" value="0.5" />
@@ -76,5 +68,4 @@
             <origin xyz="0 0 -0.15" rpy="0 0 1.57" />
             <geometry>
-<<<<<<< HEAD
                 <mesh filename="package://limo_car/meshes/limo_base.stl" scale="0.001 0.001 0.001"/>
             </geometry>
@@ -83,12 +74,4 @@
         <collision>
             <origin xyz="0 0 -0.06" rpy="0 0 0" />
-=======
-                <mesh filename="package://limo_car/meshes/limo_base.dae" scale="1 1 1"/>
-            </geometry>
-        </visual>
-        <!-- Modell für physikalische Kollision zu modellieren. -->
-        <collision>
-            <origin xyz="0 0 0" rpy="0 0 0" />
->>>>>>> origin/master
             <geometry>
                 <box size="${base_x_size} ${base_y_size} ${base_z_size}"/>
@@ -140,8 +123,5 @@
         <origin xyz="${-wheelbase/2} ${track/2} ${wheel_vertical_offset}" rpy="0 0 0" />
         <axis xyz="0 1 0"/>
-<<<<<<< HEAD
         <dynamics damping="0.1" friction="0.05"/>
-=======
->>>>>>> origin/master
     </joint>
     <link name="hinten_right_wheel_link">
@@ -170,8 +150,5 @@
         <origin xyz="${-wheelbase/2} ${-track/2} ${wheel_vertical_offset}" rpy="${M_PI} 0 0" />
         <axis xyz="0 -1 0"/>
-<<<<<<< HEAD
         <dynamics damping="0.1" friction="0.05"/>
-=======
->>>>>>> origin/master
     </joint>
     <!-- Instanziierung anderer Teile entsprechend den Makrofunktionen in "limo_anteil.xacro" -->

File: src/ros2_ws/src/limo_ros2/limo_car/urdf/limo_steering_hinge.xacro (robot description, xacro)
@@ -32,9 +32,5 @@
             <axis xyz="0 0 1" />
             <limit lower="-0.523598767" upper="0.523598767" effort="5" velocity="0.5" />
-<<<<<<< HEAD
             <dynamics damping="0.1" friction="0.05"/>
-=======
-            <dynamics damping="1.0" friction="2.0"/>
->>>>>>> origin/master
         </joint>
         <link name="front_left_wheel_link">
@@ -62,8 +58,5 @@
             <origin xyz="0 0 0" rpy="0 0 0" />
             <axis xyz="0 1 0"/>
-<<<<<<< HEAD
             <dynamics damping="0.1" friction="0.05"/>
-=======
->>>>>>> origin/master
         </joint>
     </xacro:macro>
@@ -94,9 +87,5 @@
             <axis xyz="0 0 -1"/>
             <limit lower="-0.523598767" upper="0.523598767" effort="5" velocity="0.5" />
-<<<<<<< HEAD
             <dynamics damping="0.1" friction="0.05"/>
-=======
-            <dynamics damping="1.0" friction="2.0"/>
->>>>>>> origin/master
         </joint>
         <link name="front_right_wheel_link">
@@ -124,8 +113,5 @@
             <origin xyz="0 0 0" rpy="0 0  0" />
             <axis xyz="0 -1 0"/>
-<<<<<<< HEAD
             <dynamics damping="0.1" friction="0.05"/>
-=======
->>>>>>> origin/master
         </joint>
     </xacro:macro>

File: src/ros2_ws/src/limo_ros2/limo_description/urdf/limo_ackerman.xacro (robot description, xacro)
@@ -91,8 +91,5 @@
         <origin xyz="${-wheelbase/2} ${track/2} ${wheel_vertical_offset}" rpy="0 0 0" />
         <axis xyz="0 1 0"/>
-<<<<<<< HEAD
         <dynamics damping="0.1" friction="0.05"/>
-=======
->>>>>>> origin/master
     </joint>
     <link name="rear_right_wheel_link">
@@ -122,6 +119,3 @@
         </joint>
 </robot>
-<<<<<<< HEAD
 ot>
-=======
->>>>>>> origin/master

File: src/ros2_ws/src/limo_ros2/limo_description/urdf/limo_steering_hinge.xacro (robot description, xacro)
@@ -53,8 +53,5 @@
           <origin xyz="0 0 0" rpy="0 0  0" />
           <axis xyz="0 1 0"/>
-<<<<<<< HEAD
           <dynamics damping="0.1" friction="0.05"/>
-=======
->>>>>>> origin/master
       </joint>
     </xacro:macro>
