Commit message: feat: harden pick-place pipeline — transport stability + tag-guided place dock
Fix 1 — Stop box oscillation during navigation:
  Change go_named('ready') → go_named('travel') at all three navigation-with-box
  call sites in run() so the arm is in the low-COG travel pose (joint2 tilts forward,
  arm folded down) throughout transport. Eliminates the pendulum torque on joint2.

Fix 2 — Replace unreliable blind creep with closed-loop place dock:
  navigate_to_place_table() now calls dock_to_tag() (AprilTag-guided Phase A→C→D
  controller, corrects heading regardless of Nav2 final yaw) with _dock_by_map_pos()
  fallback when the tag is not visible. Removes the 80-line 1.25 m blind creep that
  had no heading correction and drifted laterally.

Supporting changes:
  - box_pose_estimator: add /box_detection_debug image publisher with centroid
    overlay and 3D coordinate label for RViz camera panel debugging.
  - rviz/gazebo.rviz: pre-configure Box Tracker (RGB), Box Position (Marker),
    Box Pose (Arrow), and RobotModel displays so they appear by default.
  - gazebo/ackermann.xacro: fix collision mesh origin (xyz 0 0 -0.15, was -0.06 0 -0.15)
    so collision aligns with the visual mesh.
  - CMakeLists.txt: install new scripts + assets.
  - urdf/limo_ackerman_base.xacro: restore original box collision (RViz-only file,
    not used by Gazebo simulation).

Co-Authored-By: Claude Sonnet 4.6 <noreply@anthropic.com>

File: src/ros2_ws/src/limo_ros2/limo_car/gazebo/ackermann.xacro (robot description, xacro)
@@ -180,5 +180,5 @@
             <!-- Modell für physikalische Kollision zu modellieren. -->
             <collision>
-                <origin xyz="-0.06 0 -0.15" rpy="0 0 ${M_PI/2}" />
+                <origin xyz="0 0 -0.15" rpy="0 0 ${M_PI/2}" />
                 <geometry>
                     <mesh filename="package://limo_car/meshes/limo_base_collision_meters.stl" scale="1.0 1.0 1.0"/>

File: src/ros2_ws/src/limo_ros2/limo_car/urdf/limo_ackerman_base.xacro (robot description, xacro)
@@ -71,9 +71,8 @@
             </geometry>
         </visual>
-        <!-- Modell für physikalische Kollision zu modellieren. -->
         <collision>
-            <origin xyz="0 0 -0.06" rpy="0 0 0" />
+            <origin xyz="0.0 0 -0.06" rpy="0 0 0" />
             <geometry>
-                <box size="${base_x_size} ${base_y_size} ${base_z_size}"/>
+                <box size="0.32 0.20 0.12"/>
             </geometry>
         </collision>
