Commit message: feat(grasp): real physics grasp — first full six-phase pipeline pass
Replaces the kinematic weld with a contact-triggered ODE fixed joint. This is
the state that produced src/data/metrics_20260803_002247.csv:

  cycle,box_name,pick,transport,dock_via_tag,place,err_x,err_y,err_z,time_s
  0,stack_box_0,True,True,True,True,-0.0137,0.0431,-0.0001,151.96

First all-True cycle since 2026-07-02, and the first ever on a real physics
grasp rather than a kinematic weld. Faster than both 2026-07-02 baselines
(211.07 s, 193.53 s) at comparable placement error (4.5 cm vs 8.5 / 5.4 cm).

Root cause of the long-standing grasp failure: <palm_link> named 'gripper_base',
a link that does not exist in Gazebo. URDF->SDF conversion merges fixed-joint
links into their parent, so AttachObject() bailed out before ever creating the
joint. Verified with `gz model -m mbot -i`; the same bug class also invalidated
mbot::base_link and mbot::gripper_tcp.

Changes:
* gazebo_grasp_fix.cpp  — refuse to weld to STATIC models (was pinning the palm
  to ground_plane / pickup_table and locking the arm to the world)
* mycobot_ros2_control.xacro — <palm_link> gripper_base -> joint6_flange
* ackermann_with_sensor.xacro — calibrate gripper_tcp to the true grasp point
  (+0.06 m); GRASP_ABOVE 0.06 -> 0 across 7 scripts, the two cancel exactly
* nav_pick_orchestrator.py — MoveIt goal tolerance 0.025 -> 0.01 m (the old goal
  sphere was wider than the 0.035 m box); two-stage approach taking a final
  camera reading at 0.27 m instead of a single 36 cm blind drive; HOVER 0.12 ->
  0.06 with degrading fallbacks; ground-truth grasp verification
* final_map.world — pickup table raised to 0.14 m so the box enters the camera's
  vertical FOV at dock range
* grip_bench.py + grip_bench.launch.py — isolated grasp rig, ~12 s/trial vs
  ~210 s for a full cycle; resets robot and box identically each trial
* reach_sweep.py — extended grid; measured max forward reach 0.24-0.25 m

Bench result: 5/5 held, 5/5 survived wrist roll/tilt/swing (orientation coupling
the kinematic weld never had).

Co-Authored-By: Claude Opus 5 <noreply@anthropic.com>

File: src/ros2_ws/src/limo_ros2/limo_car/gazebo/ackermann_with_sensor.xacro (robot description, xacro)
@@ -59,5 +59,21 @@
     <link name="gripper_tcp"/>
     <joint name="gripper_base_to_tcp" type="fixed">
-        <origin xyz="0 0 0" rpy="0 0 0"/>
+        <!-- CALIBRATED 2026-08-01. Was xyz="0 0 0", i.e. the TCP sat on the palm and
+             the URDF admitted it: "the real fingertip offset is calibrated visually in
+             Stage 1". Stage 1 never happened, so every grasp height in the project
+             carried a hidden +0.06 correction (GRASP_ABOVE) to reach past the fingers.
+             +y is the finger axis (straight down in a top-down grasp). Two measurements
+             fix the value:
+               - TF gripper_tcp -> gripper_left1 / gripper_right1 puts the fingertip
+                 LINK midpoint at (+0.0001, +0.0255, 0) m — the knuckle line.
+               - Empirically, commanding the old TCP to (box centre + 0.060) grips the
+                 box 5/5, which means the box centre comes to rest exactly 0.060 m down
+                 the finger axis. That is the real grasp point, so that is where the TCP
+                 belongs.
+             gripper_tcp now means "the point where the box is gripped", so GRASP_ABOVE
+             drops to 0.0 everywhere. The two changes cancel exactly — the arm reaches
+             the identical physical pose — but every height in the code becomes readable
+             and the reach envelope is measured at the point that actually matters. -->
+        <origin xyz="0 0.06 0" rpy="0 0 0"/>
         <parent link="gripper_base"/>
         <child link="gripper_tcp"/>

File: src/ros2_ws/src/limo_ros2/limo_car/gazebo/mycobot_ros2_control.xacro (robot description, xacro)
@@ -116,5 +116,19 @@
   <gazebo>
     <plugin filename="libgazebo_grasp_plugin.so" name="gazebo_grasp_fix">
-      <palm_link>gripper_base</palm_link>
+      <!-- MUST be a link that exists in GAZEBO, not merely in the URDF.
+           This was 'gripper_base' and silently broke every grasp: Gazebo's URDF->SDF
+           conversion merges a link joined by a FIXED joint into its parent, so
+           gripper_base is folded into joint6_flange and disappears as an addressable
+           link (visible as joint6_flange_fixed_joint_lump__gripper_base_visual_1 in
+           `gz model -m mbot -i`). The plugin loaded fine and counted contacts fine,
+           then failed at the last step every single time:
+               [Err] [gazebo_grasp_fix.cpp:195]
+               [GazeboGraspFix] palm link 'gripper_base' not found on model
+           AttachObject() returns there WITHOUT creating the joint, so the box was
+           held by friction alone and slid out of the fingers on every lift.
+           Verified 2026-07-29 against the live model, not assumed.
+           The finger links below are fine — gripper_left1/left3/right1/right3 all
+           survive as real links because they are joined by REVOLUTE joints. -->
+      <palm_link>joint6_flange</palm_link>
       <gripper_finger_link>gripper_left1</gripper_finger_link>
       <gripper_finger_link>gripper_left3</gripper_finger_link>
